Commit message: update hardware interface

File: robotiq_ft_sensor/robotiq_ft_sensor_description/urdf/robotiq_ft300.urdf.xacro (robot description, xacro)
@@ -18,5 +18,5 @@
                 <origin xyz="0 0 0" rpy="0 0 0" />
                 <geometry>
-                    <mesh filename="file://$(find robotiq_ft_sensor_description)/meshes/visual/robotiq_ft300.STL"/>
+                    <mesh filename="package://robotiq_ft_sensor_description/meshes/visual/robotiq_ft300.STL"/>
                 </geometry>
                 <material name="Robotiq-Black">
@@ -27,5 +27,5 @@
                 <origin xyz="0 0 0" rpy="0 0 0" />
                 <geometry>
-                    <mesh filename="file://$(find robotiq_ft_sensor_description)/meshes/collision/robotiq_ft300.STL"/>
+                    <mesh filename="package://robotiq_ft_sensor_description/meshes/collision/robotiq_ft300.STL"/>
                 </geometry>
             </collision>
@@ -36,5 +36,5 @@
                 <origin xyz="0 0 0" rpy="0 0 0" />
                 <geometry>
-                    <mesh filename="file://$(find robotiq_ft_sensor_description)/meshes/visual/mountings/robotiq_ft300-G-062-COUPLING_G-50-4M6-1D6_20181119.STL"/>
+                    <mesh filename="package://robotiq_ft_sensor_description/meshes/visual/mountings/robotiq_ft300-G-062-COUPLING_G-50-4M6-1D6_20181119.STL"/>
                 </geometry>
                 <material name="Robotiq-Grey">
@@ -45,5 +45,5 @@
                 <origin xyz="0 0 0" rpy="0 0 0" />
                 <geometry>
-                    <mesh filename="file://$(find robotiq_ft_sensor_description)/meshes/collision/mountings/robotiq_ft300-G-062-COUPLING_G-50-4M6-1D6_20181119.STL"/>
+                    <mesh filename="package://robotiq_ft_sensor_description/meshes/collision/mountings/robotiq_ft300-G-062-COUPLING_G-50-4M6-1D6_20181119.STL"/>
                 </geometry>
             </collision>

File: robotiq_ft_sensor/robotiq_ft_sensor_description/urdf/robotiq_fts.ros2_control.xacro (robot description, xacro)
@@ -2,5 +2,4 @@
 <robot xmlns:xacro="http://www.ros.org/wiki/xacro">
   <xacro:macro name="robotiq_fts_ros2_control" params="
-    name
     use_fake_mode:=false
     max_retries:=1
@@ -9,5 +8,5 @@
     tf_prefix
   ">
-    <ros2_control name="${name}robotiq_ft_sensor" type="sensor">
+    <ros2_control name="${tf_prefix}robotiq_ft_sensor" type="sensor">
       <hardware>
           <plugin>robotiq_ft_sensor_hardware/RobotiqFTSensorHardware</plugin>
